File: zigbee-co2/kicad/kicad-esp32c6-co2/kicad-esp32c6-co2.kicad_sch (KiCad schematic)
At the start: 0 parts

Commit message: feat: configure PCB stackup and add custom footprint library for 4-layer board
Parts:
- added SCD41: (no value), Library:SCD41-4pins, symbol New_Library:SCD41-4pins
- added U1: XIAO-ESP32-C6-DIP, Library:XIAO-ESP32-C6-DIP, symbol seeds-studio:XIAO_ESP32-C6-DIP
Connections:
- new net: SCD41.4 (SDA), U1.5 (GPIO22/D4/SDA)
- new net: SCD41.3 (SCL), U1.6 (GPIO23/D5/SCL)
- new net +3.3V: SCD41.2 (VCC), U1.12 (3V3)
- new net GND: SCD41.1 (GND), U1.13 (GND)
- no-connect marks 0 -> 10
